File: usb_uart.kicad_sch (KiCad schematic)
At the start: 12 parts, among them U401 FT232RL, U402 CH340C

Commit message: Generate interactive bom for main and peripheral variants
Parts:
- C405, C406, C407, C409, U402: DNP (none) -> x
Changed lines of the file:
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@@
+      (effects (font (size 1.27 1.27)) hide)
+    )
+    (property "variant" "" (id 6) (at 73.66 87.63 0)
       (effects (font (size 1.27 1.27)) hide)
     )
@@
     )
     (property "PartNumber" "FT232RL" (id 5) (at 102.87 109.22 0)
+      (effects (font (size 1.27 1.27)) hide)
+    )
+    (property "variant" "" (id 6) (at 102.87 109.22 0)
       (effects (font (size 1.27 1.27)) hide)
     )
@@
       (effects (font (size 1.27 1.27)) hide)
     )
+    (property "variant" "" (id 6) (at 180.34 97.79 0)
+      (effects (font (size 1.27 1.27)) hide)
+    )
+    (property "DNP" "x" (id 7) (at 180.34 97.79 0)
+      (effects (font (size 1.27 1.27)) hide)
+    )
     (pin "1")
     (pin "10")
@@
       (effects (font (size 1.27 1.27)) hide)
     )
+    (property "variant" "" (id 6) (at 82.55 73.66 0)
+      (effects (font (size 1.27 1.27)) hide)
+    )
     (pin "1")
     (pin "2")
@@
       (effects (font (size 1.27 1.27)) hide)
     )
+    (property "variant" "" (id 6) (at 166.37 80.01 0)
+      (effects (font (size 1.27 1.27)) hide)
+    )
+    (property "DNP" "x" (id 7) (at 166.37 80.01 0)
+      (effects (font (size 1.27 1.27)) hide)
+    )
     (pin "1")
     (pin "2")
@@
       (effects (font (size 1.27 1.27)) hide)
     )
+    (property "variant" "" (id 6) (at 147.32 72.39 0)
+      (effects (font (size 1.27 1.27)) hide)
+    )
+    (property "DNP" "x" (id 7) (at 147.32 72.39 0)
+      (effects (font (size 1.27 1.27)) hide)
+    )
     (pin "1")
     (pin "2")
@@
     )
     (property "PartNumber" "Generic" (id 5) (at 135.89 72.39 0)
+      (effects (font (size 1.27 1.27)) hide)
+    )
+    (property "variant" "" (id 6) (at 135.89 72.39 0)
+      (effects (font (size 1.27 1.27)) hide)
+    )
+    (property "DNP" "x" (id 7) (at 135.89 72.39 0)
       (effects (font (size 1.27 1.27)) hide)
     )
@@
       (effects (font (size 1.27 1.27)) hide)
     )
+    (property "variant" "" (id 6) (at 157.48 72.39 0)
+      (effects (font (size 1.27 1.27)) hide)
+    )
+    (property "DNP" "x" (id 7) (at 157.48 72.39 0)
+      (effects (font (size 1.27 1.27)) hide)
+    )
     (pin "1")
     (pin "2")
@@
       (effects (font (size 1.27 1.27)) hide)
     )
+    (property "variant" "" (id 6) (at 92.71 73.66 0)
+      (effects (font (size 1.27 1.27)) hide)
+    )
     (pin "1")
     (pin "2")
@@
       (effects (font (size 1.27 1.27)) hide)
     )
+    (property "variant" "" (id 6) (at 48.26 73.66 0)
+      (effects (font (size 1.27 1.27)) hide)
+    )
     (pin "1")
     (pin "2")
@@
     )
     (property "PartNumber" "Generic" (id 5) (at 72.39 73.66 0)
+      (effects (font (size 1.27 1.27)) hide)
+    )
+    (property "variant" "" (id 6) (at 72.39 73.66 0)
       (effects (font (size 1.27 1.27)) hide)
     )
@@
       (effects (font (size 1.27 1.27)) hide)
     )
+    (property "variant" "" (id 6) (at 59.69 71.12 0)
+      (effects (font (size 1.27 1.27)) hide)
+    )
