File: digital_load.kicad_sch (KiCad schematic)
At the start: 0 parts

Commit message: WIP routing
Other:
- sheet load_control ports: added load_voltage, temp_en, temp_sense; removed none
- sheet microcontroller ports: added load_voltage, temp_en, temp_sense; removed none
