File: mcu.kicad_sch (KiCad schematic)
At the start: 16 parts

Commit message: Add heatsink, among other things
Parts:
- C10: value (none) -> 100n; footprint (none) -> Capacitor_SMD:C_0402_1005Metric
- J10: value (none) -> Conn_PIC_ICSP_ICD; footprint (none) -> Connector_PinHeader_2.54mm:PinHeader_1x06_P2.54mm_Vertical
- JP10, JP11, JP12, JP13: value (none) -> SB; footprint (none) -> Jumper:SolderJumper-2_P1.3mm_Open_TrianglePad1.0x1.5mm
- R10, R13, R14, R15, R16: value (none) -> 10k; footprint (none) -> Resistor_SMD:R_0805_2012Metric
- R11, R12, R17: value (none) -> 4.7k; footprint (none) -> Resistor_SMD:R_0805_2012Metric
- U10: value (none) -> PIC18F24K42; footprint (none) -> Package_SO:SSOP-28_5.3x10.2mm_P0.65mm
- U11: value (none) -> LM4040DBZ-2.0; footprint (none) -> Package_TO_SOT_SMD:SOT-23
Changed lines of the file:
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@@
       (effects (font (size 1.27 1.27)) (justify right))
     )
-    (property "Value" "" (id 1) (at 236.22 114.3 90)
-      (effects (font (size 1.27 1.27)) (justify right))
-    )
-    (property "Footprint" "" (id 2) (at 228.346 116.586 90)
+    (property "Value" "4.7k" (id 1) (at 236.22 114.3 90)
+      (effects (font (size 1.27 1.27)) (justify right))
+    )
+    (property "Footprint" "Resistor_SMD:R_0805_2012Metric" (id 2) (at 228.346 116.586 90)
       (effects (font (size 1.27 1.27)) hide)
     )
@@
       (effects (font (size 1.27 1.27)) (justify right))
     )
-    (property "Value" "" (id 1) (at 58.42 39.37 90)
-      (effects (font (size 1.27 1.27)) (justify right))
-    )
-    (property "Footprint" "" (id 2) (at 50.546 41.656 90)
+    (property "Value" "10k" (id 1) (at 58.42 39.37 90)
+      (effects (font (size 1.27 1.27)) (justify right))
+    )
+    (property "Footprint" "Resistor_SMD:R_0805_2012Metric" (id 2) (at 50.546 41.656 90)
       (effects (font (size 1.27 1.27)) hide)
     )
@@
       (effects (font (size 1.27 1.27)) (justify right))
     )
-    (property "Value" "" (id 1) (at 115.57 31.7499 0)
-      (effects (font (size 1.27 1.27)) (justify right))
-    )
-    (property "Footprint" "" (id 2) (at 125.73 26.67 0)
+    (property "Value" "Conn_PIC_ICSP_ICD" (id 1) (at 115.57 31.7499 0)
+      (effects (font (size 1.27 1.27)) (justify right))
+    )
+    (property "Footprint" "Connector_PinHeader_2.54mm:PinHeader_1x06_P2.54mm_Vertical" (id 2) (at 125.73 26.67 0)
       (effects (font (size 1.27 1.27)) hide)
     )
@@
     (in_bom yes) (on_board yes)
     (property "Reference" "R14" (id 0) (at 63.5 168.91 90))
-    (property "Value" "" (id 1) (at 77.47 168.91 90))
-    (property "Footprint" "" (id 2) (at 70.866 171.196 90)
+    (property "Value" "10k" (id 1) (at 77.47 168.91 90))
+    (property "Footprint" "Resistor_SMD:R_0805_2012Metric" (id 2) (at 70.866 171.196 90)
       (effects (font (size 1.27 1.27)) hide)
     )
@@
     (in_bom yes) (on_board yes)
     (property "Reference" "JP10" (id 0) (at 248.92 39.37 0))
-    (property "Value" "" (id 1) (at 242.57 36.83 0)
-      (effects (font (size 1.27 1.27)) hide)
-    )
-    (property "Footprint" "" (id 2) (at 242.57 40.64 0)
+    (property "Value" "SB" (id 1) (at 242.57 36.83 0)
+      (effects (font (size 1.27 1.27)) hide)
+    )
+    (property "Footprint" "Jumper:SolderJumper-2_P1.3mm_Open_TrianglePad1.0x1.5mm" (id 2) (at 242.57 40.64 0)
       (effects (font (size 1.27 1.27)) hide)
     )
@@
     (in_bom yes) (on_board yes)
     (property "Reference" "R15" (id 0) (at 63.5 171.45 90))
-    (property "Value" "" (id 1) (at 77.47 171.45 90))
-    (property "Footprint" "" (id 2) (at 71.374 171.704 90)
+    (property "Value" "10k" (id 1) (at 77.47 171.45 90))
+    (property "Footprint" "Resistor_SMD:R_0805_2012Metric" (id 2) (at 71.374 171.704 90)
       (effects (font (size 1.27 1.27)) hide)
     )
@@
       (effects (font (size 1.27 1.27)) (justify left))
     )
-    (property "Value" "" (id 1) (at 144.2594 77.47 0)
+    (property "Value" "PIC18F24K42" (id 1) (at 144.2594 77.47 0)
       (effects (font (size 1.27 1.27)) (justify left))
     )
-    (property "Footprint" "" (id 2) (at 125.73 115.57 0)
+    (property "Footprint" "Package_SO:SSOP-28_5.3x10.2mm_P0.65mm" (id 2) (at 125.73 115.57 0)
       (effects (font (size 1.27 1.27)) hide)
     )
@@
     (in_bom yes) (on_board yes)
     (property "Reference" "R16" (id 0) (at 63.5 177.8 90))
-    (property "Value" "" (id 1) (at 77.47 177.8 90))
-    (property "Footprint" "" (id 2) (at 70.866 180.086 90)
+    (property "Value" "10k" (id 1) (at 77.47 177.8 90))
+    (property "Footprint" "Resistor_SMD:R_0805_2012Metric" (id 2) (at 70.866 180.086 90)
       (effects (font (size 1.27 1.27)) hide)
     )
@@
       (effects (font (size 1.27 1.27)) (justify right))
     )
-    (property "Value" "" (id 1) (at 62.23 45.7199 90)
-      (effects (font (size 1.27 1.27)) (justify right))
-    )
-    (property "Footprint" "" (id 2) (at 64.77 44.45 0)
+    (property "Value" "LM4040DBZ-2.0" (id 1) (at 62.23 45.7199 90)
+      (effects (font (size 1.27 1.27)) (justify right))
+    )
+    (property "Footprint" "Package_TO_SOT_SMD:SOT-23" (id 2) (at 64.77 44.45 0)
       (effects (font (size 1.27 1.27) italic) hide)
     )
@@
       (effects (font (size 1.27 1.27)) (justify left))
     )
-    (property "Value" "" (id 1) (at 135.89 72.3962 0)
+    (property "Value" "100n" (id 1) (at 135.89 72.3962 0)
       (effects (font (size 1.27 1.27)) (justify left))
     )
-    (property "Footprint" "" (id 2) (at 133.35 71.12 0)
+    (property "Footprint" "Capacitor_SMD:C_0402_1005Metric" (id 2) (at 133.35 71.12 0)
       (effects (font (size 1.27 1.27)) hide)
     )
@@
     (in_bom yes) (on_board yes)
     (property "Reference" "R13" (id 0) (at 226.06 34.29 90))
-    (property "Value" "" (id 1) (at 228.6 34.29 90))
-    (property "Footprint" "" (id 2) (at 221.234 34.036 90)
+    (property "Value" "10k" (id 1) (at 228.6 34.29 90))
+    (property "Footprint" "Resistor_SMD:R_0805_2012Metric" (id 2) (at 221.234 34.036 90)
       (effects (font (size 1.27 1.27)) hide)
     )
@@
       (effects (font (size 1.27 1.27)) (justify right))
     )
-    (property "Value" "" (id 1) (at 236.22 111.76 90)
-      (effects (font (size 1.27 1.27)) (justify right))
-    )
-    (property "Footprint" "" (id 2) (at 228.346 114.046 90)
+    (property "Value" "4.7k" (id 1) (at 236.22 111.76 90)
+      (effects (font (size 1.27 1.27)) (justify right))
+    )
+    (property "Footprint" "Resistor_SMD:R_0805_2012Metric" (id 2) (at 228.346 114.046 90)
       (effects (font (size 1.27 1.27)) hide)
     )
@@
     (in_bom yes) (on_board yes)
     (property "Reference" "JP12" (id 0) (at 248.92 44.45 0))
-    (property "Value" "" (id 1) (at 242.57 41.91 0)
-      (effects (font (size 1.27 1.27)) hide)
-    )
-    (property "Footprint" "" (id 2) (at 242.57 45.72 0)
+    (property "Value" "SB" (id 1) (at 242.57 41.91 0)
+      (effects (font (size 1.27 1.27)) hide)
+    )
+    (property "Footprint" "Jumper:SolderJumper-2_P1.3mm_Open_TrianglePad1.0x1.5mm" (id 2) (at 242.57 45.72 0)
       (effects (font (size 1.27 1.27)) hide)
     )
@@
     (in_bom yes) (on_board yes)
     (property "Reference" "JP13" (id 0) (at 248.92 46.99 0))
-    (property "Value" "" (id 1) (at 242.57 44.45 0)
-      (effects (font (size 1.27 1.27)) hide)
-    )
-    (property "Footprint" "" (id 2) (at 242.57 48.26 0)
+    (property "Value" "SB" (id 1) (at 242.57 44.45 0)
+      (effects (font (size 1.27 1.27)) hide)
+    )
+    (property "Footprint" "Jumper:SolderJumper-2_P1.3mm_Open_TrianglePad1.0x1.5mm" (id 2) (at 242.57 48.26 0)
       (effects (font (size 1.27 1.27)) hide)
     )
@@
     (in_bom yes) (on_board yes)
     (property "Reference" "JP11" (id 0) (at 248.92 41.91 0))
-    (property "Value" "" (id 1) (at 242.57 39.37 0)
-      (effects (font (size 1.27 1.27)) hide)
-    )
-    (property "Footprint" "" (id 2) (at 242.57 43.18 0)
+    (property "Value" "SB" (id 1) (at 242.57 39.37 0)
+      (effects (font (size 1.27 1.27)) hide)
+    )
+    (property "Footprint" "Jumper:SolderJumper-2_P1.3mm_Open_TrianglePad1.0x1.5mm" (id 2) (at 242.57 43.18 0)
       (effects (font (size 1.27 1.27)) hide)
     )
@@
     (in_bom yes) (on_board yes)
     (property "Reference" "R17" (id 0) (at 63.5 180.34 90))
-    (property "Value" "" (id 1) (at 77.47 180.34 90))
-    (property "Footprint" "" (id 2) (at 71.374 180.594 90)
-      (effects (font (size 1.27 1.27)) hide)
-    )
+    (property "Value" "4.7k" (id 1) (at 77.47 180.34 90))
+    (property "Footprint" "Resistor_SMD:R_0805_2012Metric" (id 2) (at 71.374 180.594 90)
+      (effects (font (size 1.27 1.27)) hide)
+    )
