File: digital_load.kicad_pcb (KiCad board)
At the start: 4 copper layers, 50 x 50 mm, 69 parts, among them J1 Conn_01x02, J10 Conn_PIC_ICSP_ICD, J3 Conn_01x04, J4 Conn_01x04, J5 USB_C_Receptacle_USB2.0, Q20 IPA60R800CE, Q21 Q_NMOS_DGS, Q22 Q_NMOS_DGS, Q23 Q_NMOS_DGS, SW30 PEC11R, U10 PIC18F24K42, U11 LM4040DBZ-2.0, U20 LM358, U21 LM358, U30 Adafruit_PiOLED, U40 LP2951-3.3_SOIC, U60 FT232RL, U62 CH340C

Commit message: WIP routing
Parts:
- added R508: 50k, Resistor_SMD:R_0805_2012Metric, F.Cu at (144.3, 106.6)
- added TH501: Thermistor_NTC, Resistor_SMD:R_0805_2012Metric, F.Cu at (137.9, 127.5)
- Q502: renamed from Q21; value Q_NMOS_DGS -> Q_NMOS_GSD
- Q503: renamed from Q22; value Q_NMOS_DGS -> Q_NMOS_GSD
- Q504: renamed from Q23; value Q_NMOS_DGS -> Q_NMOS_GSD
- moved U502 47.1 mm to (144.2, 111.5), turned to 90 degrees
- moved R507 46.0 mm to (144.3, 116.5)
- moved C505 43.7 mm to (141.5, 109.3), turned to 90 degrees
- moved R506 41.3 mm to (144.3, 118.9), turned to 180 degrees
- moved C502 37.0 mm to (139.6, 117.4), turned to 90 degrees
- moved R503 33.6 mm to (137.0, 110.8), turned to 0 degrees
- moved U501 32.8 mm to (136.9, 115.7), turned to -90 degrees
- moved J1 32.4 mm to (107.9, 125.9)
- moved C501 32.2 mm to (133.7, 119.3)
- moved R501 32.2 mm to (127.7, 114.3)
- moved R504 30.0 mm to (137.0, 120.6), turned to 180 degrees
- moved R502 29.7 mm to (133.7, 111.5)
- moved C503 27.7 mm to (131.3, 111.5)
- moved Q504 26.6 mm to (119.2, 117.5), turned to 0 degrees
- moved C504 26.5 mm to (131.3, 115.4)
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- renumbered C10 to C301, C60 to C401, C61 to C402, C62 to C403, C63 to C404, C68 to C405, C69 to C406, C70 to C407, C20 to C501, C21 to C502, C22 to C503, C23 to C504, C24 to C505, C30 to C601, C31 to C602, C40 to C701, C41 to C702, D20 to D501, FB60 to FB401, HS20 to HS501, J5 to J2, J10 to J301, JP10 to JP301, JP11 to JP302, JP12 to JP303, JP13 to JP304, Q20 to Q501, R10 to R301, R14 to R302, R15 to R303, R16 to R304, R17 to R305, R13 to R306, R11 to R307, R12 to R308, R20 to R501, R21 to R502, R22 to R503, R29 to R504, R23 to R505, R27 to R506, R28 to R507, R24 to R509, R25 to R510, R26 to R511, R30 to R601, R31 to R602, R32 to R603, R33 to R604, R34 to R605, R40 to R701, SW30 to SW601, U11 to U301, U10 to U302, U60 to U401, U62 to U402, U20 to U501, U21 to U502, U30 to U601, U40 to U701
Connections:
- C502 pad 1: +3V3 -> +5V
- J3 pad 1: /Connectors/I2C.SCL -> /Connectors/I2C.SDA
- J3 pad 10: unconnected-(J3-Pad10) -> GND
- J3 pad 2: /Connectors/I2C.SDA -> /Connectors/I2C.SCL
- J3 pad 4: +5V -> GND
- J3 pad 5: GND -> /Connectors/load_in
- J3 pad 6: GND -> /Connectors/load_in
- J3 pad 7: unconnected-(J3-Pad7) -> /Connectors/load_in
- J3 pad 8: unconnected-(J3-Pad8) -> GND
- J3 pad 9: unconnected-(J3-Pad9) -> GND
- J301 pad 4: /microcontroller/ICSPDAT -> /microcontroller/5V_sense
- J301 pad 5: /microcontroller/ICSPCLK -> /microcontroller/3V3_sense
- J4 pad 1: /Connectors/load_in -> /Connectors/I2C.SDA
- J4 pad 2: /Connectors/load_in -> /Connectors/I2C.SCL
- J4 pad 3: /Connectors/load_in -> +5V
- J4 pad 4: /Connectors/load_in -> GND
- J4 pad 6: GND -> /Connectors/load_in
- J4 pad 7: GND -> /Connectors/load_in
- Q502 pad 1: /load_control/current_sense -> /load_control/range.1ma
- Q502 pad 2: /load_control/range.1ma -> Net-(Q502-Pad2)
- Q502 pad 3: Net-(Q21-Pad3) -> /load_control/current_sense
- Q503 pad 1: /load_control/current_sense -> /load_control/range.100ma
- Q503 pad 2: /load_control/range.100ma -> Net-(Q503-Pad2)
- Q503 pad 3: Net-(Q22-Pad3) -> /load_control/current_sense
- Q504 pad 1: /load_control/current_sense -> /load_control/range.10a
- Q504 pad 2: /load_control/range.10a -> Net-(Q504-Pad2)
- Q504 pad 3: Net-(Q23-Pad3) -> /load_control/current_sense
- R509 pad 2: Net-(Q21-Pad3) -> Net-(Q502-Pad2)
- R510 pad 2: Net-(Q22-Pad3) -> Net-(Q503-Pad2)
- R511 pad 2: Net-(Q23-Pad3) -> Net-(Q504-Pad2)
- U302 pad 16: /microcontroller/3V3_sense -> /load_control/current_measure
- U302 pad 17: /microcontroller/5V_sense -> /load_control/pwm_ctrl
- U302 pad 2: unconnected-(U10-Pad2) -> /load_control/load_voltage
- U302 pad 24: /load_control/range.100ma -> /load_control/range.1ma
- U302 pad 25: /load_control/current_measure -> /load_control/range.100ma
- U302 pad 26: /load_control/pwm_ctrl -> /load_control/range.10a
- U302 pad 27: /microcontroller/ICSPCLK -> /microcontroller/3V3_sense
- U302 pad 28: /microcontroller/ICSPDAT -> /microcontroller/5V_sense
- U302 pad 3: unconnected-(U10-Pad3) -> /load_control/temp_sense
- U302 pad 4: unconnected-(U10-Pad4) -> /load_control/temp_en
- U501 pad 8: +3V3 -> +5V
- U502 pad 5: unconnected-(U21-Pad5) -> Net-(R508-Pad2)
- U502 pad 6: unconnected-(U21-Pad6) -> /load_control/temp_sense
- U502 pad 7: unconnected-(U21-Pad7) -> /load_control/temp_sense
Routing:
- net /microcontroller/~{MCLR}/VPP: track 0.00 -> 29.0 mm, vias 0 -> 1
- net /load_control/current_sense: track 4.05 -> 32.7 mm
- net Net-(R508-Pad2): track 0.00 -> 25.9 mm
- net /microcontroller/5V_sense: track 12.0 -> 34.8 mm, vias 0 -> 2
- net /load_control/load_voltage: track 0.00 -> 20.0 mm
- net /load_control/temp_sense: track 0.00 -> 19.4 mm
- net /load_control/pwm_ctrl: track 0.00 -> 17.7 mm
- net /load_control/temp_en: track 0.00 -> 17.4 mm
- net /microcontroller/3V3_sense: track 16.1 -> 32.8 mm, vias 0 -> 2
- net /load_control/range.1ma: track 0.00 -> 15.6 mm
- net /load_control/current_measure: track 19.1 -> 34.0 mm, vias 0 -> 2
- net GND: track 51.0 -> 65.3 mm, vias 18 -> 27
- net /load_control/range.10a: track 0.00 -> 14.1 mm
- net /load_control/range.100ma: track 0.00 -> 12.3 mm
- net /Display_Encoder/ENC.A: track 15.1 -> 6.60 mm
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- added copper zone on In2.Cu, net /Connectors/load_in

Commit message: Routing almost complete
Parts:
- moved C405 2.93 mm to (113.1, 125.8)
- moved C404 1.97 mm to (116.2, 108.9)
- moved C406 1.41 mm to (113.6, 123.8), turned to 180 degrees
- moved U402 1.04 mm to (109.6, 119.2)
- moved C407 0.78 mm to (110.3, 114.1), turned to 90 degrees
Routing:
- net /Connectors/I2C.SDA: track 20.9 -> 84.5 mm, vias 1 -> 2
- net /Connectors/I2C.SCL: track 24.7 -> 84.8 mm
- net /microcontroller/UART.RTS: track 17.1 -> 33.0 mm
- net Net-(Q501-Pad1): track 3.21 -> 14.1 mm, vias 0 -> 2
- net /microcontroller/UART.RX: track 7.91 -> 17.6 mm
- net /microcontroller/UART.CTS: track 15.2 -> 24.5 mm, vias 1 -> 0
- net /microcontroller/UART.TX: track 13.9 -> 21.5 mm, vias 0 -> 2
- net Net-(C401-Pad1): track 14.4 -> 12.4 mm, vias 4 -> 3
- net /Connectors/load_in: track 0.00 -> 1.35 mm, vias 0 -> 1
- net GND: track 65.3 -> 66.3 mm, vias 27 -> 26
- net /Connectors/USB2.0.D-: track 37.4 -> 38.4 mm
- net /Connectors/USB2.0.D+: track 36.6 -> 37.7 mm
- added copper zone on In2.Cu, net +3V3
- added copper zone on In2.Cu, net +5V
- added copper zone on B.Cu, net /Connectors/load_in
- added copper zone on In2.Cu, net Net-(C401-Pad1)
- removed copper zone on In2.Cu, net /Connectors/load_in
