File: connectors.kicad_sch (KiCad schematic)
At the start: 7 parts, among them J1 Conn_01x02, J2 USB_C_Receptacle_USB2.0, J3 Conn_01x04, J4 Conn_01x04

Commit message: Add partnumbers
Parts:
- D1: value SP0503BAHT -> (none); footprint Package_TO_SOT_SMD:SOT-143 -> (none); Manufacturer (none) -> Littlefuse; PartNumber (none) -> SP0503BAHTG
- J1: value Conn_01x02 -> (none); footprint Connector_PinHeader_2.54mm:PinHeader_1x02_P2.54mm_Horizontal -> (none); Manufacturer (none) -> Generic; PartNumber (none) -> Generic
- J2: value USB_C_Receptacle_USB2.0 -> (none); footprint Connector_USB:USB_C_Receptacle_GCT_USB4085 -> (none); Manufacturer (none) -> GCT; PartNumber (none) -> USB4085
- J3, J4: value Conn_01x04 -> (none); footprint Connector_PinSocket_2.54mm:PinSocket_1x10_P2.54mm_Vertical -> (none); Manufacturer (none) -> Generic; PartNumber (none) -> Generic
- R1, R2: value 5.1k -> (none); footprint Resistor_SMD:R_0805_2012Metric -> (none); Manufacturer (none) -> Generic; PartNumber (none) -> Generic
Changed lines of the file:
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@@
     (in_bom yes) (on_board yes) (fields_autoplaced)
     (property "Reference" "J3" (id 0) (at 168.91 45.72 0))
-    (property "Value" "Conn_01x04" (id 1) (at 168.91 48.26 0))
-    (property "Footprint" "Connector_PinSocket_2.54mm:PinSocket_1x10_P2.54mm_Vertical" (id 2) (at 168.91 62.23 0)
+    (property "Value" "" (id 1) (at 168.91 48.26 0))
+    (property "Footprint" "" (id 2) (at 168.91 62.23 0)
       (effects (font (size 1.27 1.27)) hide)
     )
     (property "Datasheet" "~" (id 3) (at 168.91 62.23 0)
+      (effects (font (size 1.27 1.27)) hide)
+    )
+    (property "Manufacturer" "Generic" (id 4) (at 168.91 62.23 0)
+      (effects (font (size 1.27 1.27)) hide)
+    )
+    (property "PartNumber" "Generic" (id 5) (at 168.91 62.23 0)
       (effects (font (size 1.27 1.27)) hide)
     )
@@
     (in_bom no) (on_board yes)
     (property "Reference" "R1" (id 0) (at 76.2 140.97 90))
-    (property "Value" "5.1k" (id 1) (at 76.2 130.81 90))
-    (property "Footprint" "Resistor_SMD:R_0805_2012Metric" (id 2) (at 76.454 135.636 90)
+    (property "Value" "" (id 1) (at 76.2 130.81 90))
+    (property "Footprint" "" (id 2) (at 76.454 135.636 90)
       (effects (font (size 1.27 1.27)) hide)
     )
@@
       (effects (font (size 1.27 1.27)) hide)
     )
+    (property "Manufacturer" "Generic" (id 4) (at 77.47 135.89 0)
+      (effects (font (size 1.27 1.27)) hide)
+    )
+    (property "PartNumber" "Generic" (id 5) (at 77.47 135.89 0)
+      (effects (font (size 1.27 1.27)) hide)
+    )
     (pin "1")
     (pin "2")
@@
     (in_bom yes) (on_board yes) (fields_autoplaced)
     (property "Reference" "J1" (id 0) (at 36.83 41.91 0))
-    (property "Value" "Conn_01x02" (id 1) (at 36.83 44.45 0))
-    (property "Footprint" "Connector_PinHeader_2.54mm:PinHeader_1x02_P2.54mm_Horizontal" (id 2) (at 36.83 48.26 0)
+    (property "Value" "" (id 1) (at 36.83 44.45 0))
+    (property "Footprint" "" (id 2) (at 36.83 48.26 0)
       (effects (font (size 1.27 1.27)) hide)
     )
     (property "Datasheet" "~" (id 3) (at 36.83 48.26 0)
+      (effects (font (size 1.27 1.27)) hide)
+    )
+    (property "Manufacturer" "Generic" (id 4) (at 36.83 48.26 0)
+      (effects (font (size 1.27 1.27)) hide)
+    )
+    (property "PartNumber" "Generic" (id 5) (at 36.83 48.26 0)
       (effects (font (size 1.27 1.27)) hide)
     )
@@
     (in_bom no) (on_board yes)
     (property "Reference" "R2" (id 0) (at 80.01 140.97 90))
-    (property "Value" "5.1k" (id 1) (at 80.01 130.81 90))
-    (property "Footprint" "Resistor_SMD:R_0805_2012Metric" (id 2) (at 80.264 135.636 90)
+    (property "Value" "" (id 1) (at 80.01 130.81 90))
+    (property "Footprint" "" (id 2) (at 80.264 135.636 90)
       (effects (font (size 1.27 1.27)) hide)
     )
     (property "Datasheet" "~" (id 3) (at 81.28 135.89 0)
+      (effects (font (size 1.27 1.27)) hide)
+    )
+    (property "Manufacturer" "Generic" (id 4) (at 81.28 135.89 0)
+      (effects (font (size 1.27 1.27)) hide)
+    )
+    (property "PartNumber" "Generic" (id 5) (at 81.28 135.89 0)
       (effects (font (size 1.27 1.27)) hide)
     )
@@
     (in_bom yes) (on_board yes) (fields_autoplaced)
     (property "Reference" "J2" (id 0) (at 45.72 90.17 0))
-    (property "Value" "USB_C_Receptacle_USB2.0" (id 1) (at 45.72 92.71 0))
-    (property "Footprint" "Connector_USB:USB_C_Receptacle_GCT_USB4085" (id 2) (at 49.53 113.03 0)
+    (property "Value" "" (id 1) (at 45.72 92.71 0))
+    (property "Footprint" "" (id 2) (at 49.53 113.03 0)
       (effects (font (size 1.27 1.27)) hide)
     )
     (property "Datasheet" "https://www.usb.org/sites/default/files/documents/usb_type-c.zip" (id 3) (at 49.53 113.03 0)
+      (effects (font (size 1.27 1.27)) hide)
+    )
+    (property "Manufacturer" "GCT" (id 4) (at 45.72 113.03 0)
+      (effects (font (size 1.27 1.27)) hide)
+    )
+    (property "PartNumber" "USB4085" (id 5) (at 45.72 113.03 0)
       (effects (font (size 1.27 1.27)) hide)
     )
@@
       (effects (font (size 1.27 1.27)) (justify left))
     )
-    (property "Value" "Conn_01x04" (id 1) (at 267.97 64.7699 0)
+    (property "Value" "" (id 1) (at 267.97 64.7699 0)
       (effects (font (size 1.27 1.27)) (justify left))
     )
-    (property "Footprint" "Connector_PinSocket_2.54mm:PinSocket_1x10_P2.54mm_Vertical" (id 2) (at 265.43 62.23 0)
+    (property "Footprint" "" (id 2) (at 265.43 62.23 0)
       (effects (font (size 1.27 1.27)) hide)
     )
     (property "Datasheet" "~" (id 3) (at 265.43 62.23 0)
+      (effects (font (size 1.27 1.27)) hide)
+    )
+    (property "Manufacturer" "Generic" (id 4) (at 265.43 62.23 0)
+      (effects (font (size 1.27 1.27)) hide)
+    )
+    (property "PartNumber" "Generic" (id 5) (at 265.43 62.23 0)
       (effects (font (size 1.27 1.27)) hide)
     )
@@
       (effects (font (size 1.27 1.27)) (justify left))
     )
-    (property "Value" "SP0503BAHT" (id 1) (at 73.66 125.7299 0)
+    (property "Value" "" (id 1) (at 73.66 125.7299 0)
       (effects (font (size 1.27 1.27)) (justify left))
     )
-    (property "Footprint" "Package_TO_SOT_SMD:SOT-143" (id 2) (at 73.025 125.73 0)
+    (property "Footprint" "" (id 2) (at 73.025 125.73 0)
       (effects (font (size 1.27 1.27)) (justify left) hide)
     )
@@
       (effects (font (size 1.27 1.27)) hide)
     )
+    (property "Manufacturer" "Littlefuse" (id 4) (at 67.31 124.46 0)
+      (effects (font (size 1.27 1.27)) hide)
+    )
+    (property "PartNumber" "SP0503BAHTG" (id 5) (at 67.31 124.46 0)
+      (effects (font (size 1.27 1.27)) hide)
+    )

Commit message: Fix missing footprints in schematic
Parts:
- J1, J3, J4: now left out of the parts list
Changed lines of the file:
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@@
   )
   (symbol (lib_id "Connector_Generic:Conn_01x10") (at 168.91 62.23 0) (mirror y) (unit 1)
-    (in_bom yes) (on_board yes) (fields_autoplaced)
+    (in_bom no) (on_board yes) (fields_autoplaced)
     (property "Reference" "J3" (id 0) (at 168.91 45.72 0))
     (property "Value" "" (id 1) (at 168.91 48.26 0))
@@
   )
   (symbol (lib_id "Connector_Generic:Conn_01x02") (at 36.83 48.26 0) (mirror y) (unit 1)
-    (in_bom yes) (on_board yes) (fields_autoplaced)
+    (in_bom no) (on_board yes) (fields_autoplaced)
     (property "Reference" "J1" (id 0) (at 36.83 41.91 0))
     (property "Value" "" (id 1) (at 36.83 44.45 0))
@@
   )
   (symbol (lib_id "Connector_Generic:Conn_01x10") (at 265.43 62.23 0) (unit 1)
-    (in_bom yes) (on_board yes) (fields_autoplaced)
+    (in_bom no) (on_board yes) (fields_autoplaced)
     (property "Reference" "J4" (id 0) (at 267.97 62.2299 0)
       (effects (font (size 1.27 1.27)) (justify left))

Commit message: Reduce trace resistance of 10mOhm channel
Parts:
- D1: value (none) -> SP0503BAHTG; footprint (none) -> Package_TO_SOT_SMD:SOT-143
- J1: value (none) -> Conn_01x02; footprint (none) -> Connector_PinHeader_2.54mm:PinHeader_1x02_P2.54mm_Horizontal
- J2: value (none) -> USB_C_Receptacle_USB2.0; footprint (none) -> Connector_USB:USB_C_Receptacle_GCT_USB4085
- J3, J4: value (none) -> Conn_01x10; footprint (none) -> Connector_PinSocket_2.54mm:PinSocket_1x10_P2.54mm_Vertical
- R1, R2: value (none) -> 5.1k; footprint (none) -> Resistor_SMD:R_0805_2012Metric
Changed lines of the file:
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@@
     (in_bom no) (on_board yes) (fields_autoplaced)
     (property "Reference" "J3" (id 0) (at 168.91 45.72 0))
-    (property "Value" "" (id 1) (at 168.91 48.26 0))
-    (property "Footprint" "" (id 2) (at 168.91 62.23 0)
+    (property "Value" "Conn_01x10" (id 1) (at 168.91 48.26 0))
+    (property "Footprint" "Connector_PinSocket_2.54mm:PinSocket_1x10_P2.54mm_Vertical" (id 2) (at 168.91 62.23 0)
       (effects (font (size 1.27 1.27)) hide)
     )
@@
     (in_bom no) (on_board yes)
     (property "Reference" "R1" (id 0) (at 76.2 140.97 90))
-    (property "Value" "" (id 1) (at 76.2 130.81 90))
-    (property "Footprint" "" (id 2) (at 76.454 135.636 90)
+    (property "Value" "5.1k" (id 1) (at 76.2 130.81 90))
+    (property "Footprint" "Resistor_SMD:R_0805_2012Metric" (id 2) (at 76.454 135.636 90)
       (effects (font (size 1.27 1.27)) hide)
     )
@@
     (in_bom no) (on_board yes) (fields_autoplaced)
     (property "Reference" "J1" (id 0) (at 36.83 41.91 0))
-    (property "Value" "" (id 1) (at 36.83 44.45 0))
-    (property "Footprint" "" (id 2) (at 36.83 48.26 0)
+    (property "Value" "Conn_01x02" (id 1) (at 36.83 44.45 0))
+    (property "Footprint" "Connector_PinHeader_2.54mm:PinHeader_1x02_P2.54mm_Horizontal" (id 2) (at 36.83 48.26 0)
       (effects (font (size 1.27 1.27)) hide)
     )
@@
     (in_bom no) (on_board yes)
     (property "Reference" "R2" (id 0) (at 80.01 140.97 90))
-    (property "Value" "" (id 1) (at 80.01 130.81 90))
-    (property "Footprint" "" (id 2) (at 80.264 135.636 90)
+    (property "Value" "5.1k" (id 1) (at 80.01 130.81 90))
+    (property "Footprint" "Resistor_SMD:R_0805_2012Metric" (id 2) (at 80.264 135.636 90)
       (effects (font (size 1.27 1.27)) hide)
     )
@@
     (in_bom yes) (on_board yes) (fields_autoplaced)
     (property "Reference" "J2" (id 0) (at 45.72 90.17 0))
-    (property "Value" "" (id 1) (at 45.72 92.71 0))
-    (property "Footprint" "" (id 2) (at 49.53 113.03 0)
+    (property "Value" "USB_C_Receptacle_USB2.0" (id 1) (at 45.72 92.71 0))
+    (property "Footprint" "Connector_USB:USB_C_Receptacle_GCT_USB4085" (id 2) (at 49.53 113.03 0)
       (effects (font (size 1.27 1.27)) hide)
     )
@@
       (effects (font (size 1.27 1.27)) (justify left))
     )
-    (property "Value" "" (id 1) (at 267.97 64.7699 0)
+    (property "Value" "Conn_01x10" (id 1) (at 267.97 64.7699 0)
       (effects (font (size 1.27 1.27)) (justify left))
     )
-    (property "Footprint" "" (id 2) (at 265.43 62.23 0)
+    (property "Footprint" "Connector_PinSocket_2.54mm:PinSocket_1x10_P2.54mm_Vertical" (id 2) (at 265.43 62.23 0)
       (effects (font (size 1.27 1.27)) hide)
     )
@@
       (effects (font (size 1.27 1.27)) (justify left))
     )
-    (property "Value" "" (id 1) (at 73.66 125.7299 0)
+    (property "Value" "SP0503BAHTG" (id 1) (at 73.66 125.7299 0)
       (effects (font (size 1.27 1.27)) (justify left))
     )
-    (property "Footprint" "" (id 2) (at 73.025 125.73 0)
+    (property "Footprint" "Package_TO_SOT_SMD:SOT-143" (id 2) (at 73.025 125.73 0)
       (effects (font (size 1.27 1.27)) (justify left) hide)
     )

Commit message: Generate interactive bom for main and peripheral variants
Parts:
- D1, J1, J2, R1, R2: variant (none) -> main_only
Changed lines of the file:
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@@
+      (effects (font (size 1.27 1.27)) hide)
+    )
+    (property "variant" "" (id 6) (at 168.91 62.23 0)
       (effects (font (size 1.27 1.27)) hide)
     )
@@
       (effects (font (size 1.27 1.27)) hide)
     )
+    (property "variant" "main_only" (id 6) (at 77.47 135.89 0)
+      (effects (font (size 1.27 1.27)) hide)
+    )
     (pin "1")
     (pin "2")
@@
       (effects (font (size 1.27 1.27)) hide)
     )
+    (property "variant" "main_only" (id 6) (at 36.83 48.26 0)
+      (effects (font (size 1.27 1.27)) hide)
+    )
     (pin "1")
     (pin "2")
@@
       (effects (font (size 1.27 1.27)) hide)
     )
+    (property "variant" "main_only" (id 6) (at 81.28 135.89 0)
+      (effects (font (size 1.27 1.27)) hide)
+    )
     (pin "1")
     (pin "2")
@@
     )
     (property "PartNumber" "USB4085" (id 5) (at 45.72 113.03 0)
+      (effects (font (size 1.27 1.27)) hide)
+    )
+    (property "variant" "main_only" (id 6) (at 45.72 113.03 0)
       (effects (font (size 1.27 1.27)) hide)
     )
@@
       (effects (font (size 1.27 1.27)) hide)
     )
+    (property "variant" "" (id 6) (at 265.43 62.23 0)
+      (effects (font (size 1.27 1.27)) hide)
+    )
     (pin "1")
     (pin "10")
@@
       (effects (font (size 1.27 1.27)) hide)
     )
+    (property "variant" "main_only" (id 6) (at 67.31 124.46 0)
+      (effects (font (size 1.27 1.27)) hide)
+    )
