File: display_encoder.kicad_sch (KiCad schematic)
At the start: 9 parts

Commit message: Fix missing footprints in schematic
Parts:
- C601, C602, R601, R602, R603, R604, R605: now left out of the parts list
Changed lines of the file:
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@@
   )
   (symbol (lib_id "Device:R_US") (at 149.86 69.85 90) (unit 1)
-    (in_bom yes) (on_board yes)
+    (in_bom no) (on_board yes)
     (property "Reference" "R601" (id 0) (at 149.86 73.66 90))
     (property "Value" "" (id 1) (at 149.86 76.2 90))
@@
   )
   (symbol (lib_id "Device:C") (at 137.16 73.66 180) (unit 1)
-    (in_bom yes) (on_board yes) (fields_autoplaced)
+    (in_bom no) (on_board yes) (fields_autoplaced)
     (property "Reference" "C601" (id 0) (at 140.97 72.3899 0)
       (effects (font (size 1.27 1.27)) (justify right))
@@
   )
   (symbol (lib_id "Device:C") (at 137.16 91.44 180) (unit 1)
-    (in_bom yes) (on_board yes) (fields_autoplaced)
+    (in_bom no) (on_board yes) (fields_autoplaced)
     (property "Reference" "C602" (id 0) (at 140.97 90.1699 0)
       (effects (font (size 1.27 1.27)) (justify right))
@@
   )
   (symbol (lib_id "Device:R_US") (at 153.67 66.04 0) (unit 1)
-    (in_bom yes) (on_board yes)
+    (in_bom no) (on_board yes)
     (property "Reference" "R603" (id 0) (at 147.32 66.04 90))
     (property "Value" "" (id 1) (at 149.86 66.04 90))
@@
   )
   (symbol (lib_id "Device:R_US") (at 180.34 69.85 180) (unit 1)
-    (in_bom yes) (on_board yes)
+    (in_bom no) (on_board yes)
     (property "Reference" "R605" (id 0) (at 184.15 69.85 90))
     (property "Value" "" (id 1) (at 186.69 69.85 90))
@@
   )
   (symbol (lib_id "Device:R_US") (at 149.86 87.63 90) (unit 1)
-    (in_bom yes) (on_board yes)
+    (in_bom no) (on_board yes)
     (property "Reference" "R602" (id 0) (at 149.86 91.44 90))
     (property "Value" "" (id 1) (at 149.86 93.98 90))
@@
   )
   (symbol (lib_id "Device:R_US") (at 158.75 66.04 180) (unit 1)
-    (in_bom yes) (on_board yes)
+    (in_bom no) (on_board yes)
     (property "Reference" "R604" (id 0) (at 162.56 66.04 90))
     (property "Value" "" (id 1) (at 165.1 66.04 90))

Commit message: Reduce trace resistance of 10mOhm channel
Parts:
- C601, C602: value (none) -> 10n; footprint (none) -> Capacitor_SMD:C_0805_2012Metric
- R601, R602, R603, R604, R605: value (none) -> 10k; footprint (none) -> Resistor_SMD:R_0805_2012Metric
- SW601: value (none) -> PEC11R; footprint (none) -> Rotary_Encoder:RotaryEncoder_Alps_EC12E-Switch_Vertical_H20mm
- U601: value (none) -> Adafruit_PiOLED; footprint (none) -> 0_Display:PiOLED
Changed lines of the file:
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@@
     (in_bom no) (on_board yes)
     (property "Reference" "R601" (id 0) (at 149.86 73.66 90))
-    (property "Value" "" (id 1) (at 149.86 76.2 90))
-    (property "Footprint" "" (id 2) (at 150.114 68.834 90)
+    (property "Value" "10k" (id 1) (at 149.86 76.2 90))
+    (property "Footprint" "Resistor_SMD:R_0805_2012Metric" (id 2) (at 150.114 68.834 90)
       (effects (font (size 1.27 1.27)) hide)
     )
@@
     (in_bom yes) (on_board yes) (fields_autoplaced)
     (property "Reference" "U601" (id 0) (at 161.29 116.84 0))
-    (property "Value" "" (id 1) (at 161.29 119.38 0))
-    (property "Footprint" "" (id 2) (at 162.56 121.92 0)
+    (property "Value" "Adafruit_PiOLED" (id 1) (at 161.29 119.38 0))
+    (property "Footprint" "0_Display:PiOLED" (id 2) (at 162.56 121.92 0)
       (effects (font (size 1.27 1.27)) hide)
     )
@@
       (effects (font (size 1.27 1.27)) (justify right))
     )
-    (property "Value" "" (id 1) (at 140.97 74.9299 0)
-      (effects (font (size 1.27 1.27)) (justify right))
-    )
-    (property "Footprint" "" (id 2) (at 136.1948 69.85 0)
+    (property "Value" "10n" (id 1) (at 140.97 74.9299 0)
+      (effects (font (size 1.27 1.27)) (justify right))
+    )
+    (property "Footprint" "Capacitor_SMD:C_0805_2012Metric" (id 2) (at 136.1948 69.85 0)
       (effects (font (size 1.27 1.27)) hide)
     )
@@
     (in_bom yes) (on_board yes)
     (property "Reference" "SW601" (id 0) (at 170.18 68.58 0))
-    (property "Value" "" (id 1) (at 170.18 71.12 0))
-    (property "Footprint" "" (id 2) (at 166.37 74.676 0)
+    (property "Value" "PEC11R" (id 1) (at 170.18 71.12 0))
+    (property "Footprint" "Rotary_Encoder:RotaryEncoder_Alps_EC12E-Switch_Vertical_H20mm" (id 2) (at 166.37 74.676 0)
       (effects (font (size 1.27 1.27)) hide)
     )
@@
       (effects (font (size 1.27 1.27)) (justify right))
     )
-    (property "Value" "" (id 1) (at 140.97 92.7099 0)
-      (effects (font (size 1.27 1.27)) (justify right))
-    )
-    (property "Footprint" "" (id 2) (at 136.1948 87.63 0)
+    (property "Value" "10n" (id 1) (at 140.97 92.7099 0)
+      (effects (font (size 1.27 1.27)) (justify right))
+    )
+    (property "Footprint" "Capacitor_SMD:C_0805_2012Metric" (id 2) (at 136.1948 87.63 0)
       (effects (font (size 1.27 1.27)) hide)
     )
@@
     (in_bom no) (on_board yes)
     (property "Reference" "R603" (id 0) (at 147.32 66.04 90))
-    (property "Value" "" (id 1) (at 149.86 66.04 90))
-    (property "Footprint" "" (id 2) (at 154.686 66.294 90)
+    (property "Value" "10k" (id 1) (at 149.86 66.04 90))
+    (property "Footprint" "Resistor_SMD:R_0805_2012Metric" (id 2) (at 154.686 66.294 90)
       (effects (font (size 1.27 1.27)) hide)
     )
@@
     (in_bom no) (on_board yes)
     (property "Reference" "R605" (id 0) (at 184.15 69.85 90))
-    (property "Value" "" (id 1) (at 186.69 69.85 90))
-    (property "Footprint" "" (id 2) (at 179.324 69.596 90)
+    (property "Value" "10k" (id 1) (at 186.69 69.85 90))
+    (property "Footprint" "Resistor_SMD:R_0805_2012Metric" (id 2) (at 179.324 69.596 90)
       (effects (font (size 1.27 1.27)) hide)
     )
@@
     (in_bom no) (on_board yes)
     (property "Reference" "R602" (id 0) (at 149.86 91.44 90))
-    (property "Value" "" (id 1) (at 149.86 93.98 90))
-    (property "Footprint" "" (id 2) (at 150.114 86.614 90)
+    (property "Value" "10k" (id 1) (at 149.86 93.98 90))
+    (property "Footprint" "Resistor_SMD:R_0805_2012Metric" (id 2) (at 150.114 86.614 90)
       (effects (font (size 1.27 1.27)) hide)
     )
@@
     (in_bom no) (on_board yes)
     (property "Reference" "R604" (id 0) (at 162.56 66.04 90))
-    (property "Value" "" (id 1) (at 165.1 66.04 90))
-    (property "Footprint" "" (id 2) (at 157.734 65.786 90)
-      (effects (font (size 1.27 1.27)) hide)
-    )
+    (property "Value" "10k" (id 1) (at 165.1 66.04 90))
+    (property "Footprint" "Resistor_SMD:R_0805_2012Metric" (id 2) (at 157.734 65.786 90)
+      (effects (font (size 1.27 1.27)) hide)
+    )

Commit message: Generate interactive bom for main and peripheral variants
Parts:
- C601, C602, R601, R602, R603, R604, R605, SW601, U601: variant (none) -> main_only
Changed lines of the file:
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@@
+      (effects (font (size 1.27 1.27)) hide)
+    )
+    (property "variant" "main_only" (id 6) (at 149.86 69.85 0)
       (effects (font (size 1.27 1.27)) hide)
     )
@@
     )
     (property "PartNumber" "PiOled" (id 5) (at 161.29 127 0)
+      (effects (font (size 1.27 1.27)) hide)
+    )
+    (property "variant" "main_only" (id 6) (at 161.29 127 0)
       (effects (font (size 1.27 1.27)) hide)
     )
@@
     )
     (property "PartNumber" "Generic" (id 5) (at 137.16 73.66 0)
+      (effects (font (size 1.27 1.27)) hide)
+    )
+    (property "variant" "main_only" (id 6) (at 137.16 73.66 0)
       (effects (font (size 1.27 1.27)) hide)
     )
@@
       (effects (font (size 1.27 1.27)) hide)
     )
+    (property "variant" "main_only" (id 6) (at 170.18 78.74 0)
+      (effects (font (size 1.27 1.27)) hide)
+    )
     (pin "A")
     (pin "B")
@@
       (effects (font (size 1.27 1.27)) hide)
     )
+    (property "variant" "main_only" (id 6) (at 137.16 91.44 0)
+      (effects (font (size 1.27 1.27)) hide)
+    )
     (pin "1")
     (pin "2")
@@
       (effects (font (size 1.27 1.27)) hide)
     )
+    (property "variant" "main_only" (id 6) (at 153.67 66.04 0)
+      (effects (font (size 1.27 1.27)) hide)
+    )
     (pin "1")
     (pin "2")
@@
       (effects (font (size 1.27 1.27)) hide)
     )
+    (property "variant" "main_only" (id 6) (at 180.34 69.85 0)
+      (effects (font (size 1.27 1.27)) hide)
+    )
     (pin "1")
     (pin "2")
@@
       (effects (font (size 1.27 1.27)) hide)
     )
+    (property "variant" "main_only" (id 6) (at 149.86 87.63 0)
+      (effects (font (size 1.27 1.27)) hide)
+    )
     (pin "1")
     (pin "2")
@@
       (effects (font (size 1.27 1.27)) hide)
     )
+    (property "variant" "main_only" (id 6) (at 158.75 66.04 0)
+      (effects (font (size 1.27 1.27)) hide)
+    )
