File: load_control.kicad_sch (KiCad schematic)
At the start: 25 parts

Commit message: Reduce trace resistance of 10mOhm channel
Parts:
- C501: value (none) -> 4.7u; footprint (none) -> Capacitor_SMD:C_0805_2012Metric
- C502, C505: value (none) -> 100n; footprint (none) -> Capacitor_SMD:C_0402_1005Metric
- C503, C504: value (none) -> 10n; footprint (none) -> Capacitor_SMD:C_0805_2012Metric
- D501: value (none) -> DIODE; footprint (none) -> Diode_SMD:D_SOD-323
- HS501: value (none) -> Heatsink_Pad; footprint (none) -> 0_Heatsink:Heatsink_ASSMANN_WSW_V6560W
- Q501: value (none) -> IRLS640A; footprint (none) -> Package_TO_SOT_THT:TO-220-3_Vertical
- Q502, Q503, Q504: value (none) -> Q_NMOS_GSD; footprint (none) -> Package_TO_SOT_SMD:SOT-23
- R501, R503, R504, R505, R508: value (none) -> 10k; footprint (none) -> Resistor_SMD:R_0805_2012Metric
- R502: value (none) -> 270k; footprint (none) -> Resistor_SMD:R_0805_2012Metric
- R506: value (none) -> 4.7M; footprint (none) -> Resistor_SMD:R_0805_2012Metric
- R507: value (none) -> 47k; footprint (none) -> Resistor_SMD:R_0805_2012Metric
- R509: value (none) -> 100; footprint (none) -> Resistor_SMD:R_0805_2012Metric
- R510: value (none) -> 1; footprint (none) -> Resistor_SMD:R_0805_2012Metric
- R511: value (none) -> 10m; footprint (none) -> Resistor_SMD:R_0805_2012Metric
- TH501: value (none) -> Thermistor_NTC; footprint (none) -> Resistor_SMD:R_0402_1005Metric
- U501, U502: value (none) -> LM2904BA; footprint (none) -> Package_SO:TSSOP-8_4.4x3mm_P0.65mm
Connections:
- net at R509.2: now also Q504.2 (S); no longer Q502.2 (S)
- net at R511.2: now also Q502.2 (S); no longer Q504.2 (S)
Other:
- moved on the sheet: R509, R511
