File: power.kicad_sch (KiCad schematic)
At the start: 6 parts

Commit message: Change some partnumbers in preparation for the order
Parts:
- U701: PartNumber LP2951-33D -> LP2951-30D
Changed lines of the file:
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@@
   (symbol (lib_id "power:GND") (at 172.72 81.28 0) (unit 1)
     (in_bom yes) (on_board yes) (fields_autoplaced)
-    (property "Reference" "#PWR?" (id 0) (at 172.72 87.63 0)
+    (property "Reference" "#PWR0103" (id 0) (at 172.72 87.63 0)
       (effects (font (size 1.27 1.27)) hide)
     )
@@
       (effects (font (size 1.27 1.27)) hide)
     )
-    (property "PartNumber" "LP2951-33D" (id 5) (at 154.94 71.12 0)
+    (property "PartNumber" "LP2951-30D" (id 5) (at 154.94 71.12 0)
       (effects (font (size 1.27 1.27)) hide)
     )

Commit message: Reduce trace resistance of 10mOhm channel
Parts:
- C701, C702: value (none) -> 1u; footprint (none) -> Capacitor_SMD:C_0805_2012Metric
- R701: value (none) -> 10k; footprint (none) -> Resistor_SMD:R_0805_2012Metric
- R702: value (none) -> 200k; footprint (none) -> Resistor_SMD:R_0805_2012Metric
- R703: value (none) -> 120k; footprint (none) -> Resistor_SMD:R_0805_2012Metric
- U701: value (none) -> LP2951-3.3_SOIC; footprint (none) -> Package_SO:SOIC-8_3.9x4.9mm_P1.27mm
Changed lines of the file:
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@@
       (effects (font (size 1.27 1.27)) (justify left))
     )
-    (property "Value" "" (id 1) (at 184.15 68.5799 0)
+    (property "Value" "1u" (id 1) (at 184.15 68.5799 0)
       (effects (font (size 1.27 1.27)) (justify left))
     )
-    (property "Footprint" "" (id 2) (at 181.3052 71.12 0)
+    (property "Footprint" "Capacitor_SMD:C_0805_2012Metric" (id 2) (at 181.3052 71.12 0)
       (effects (font (size 1.27 1.27)) hide)
     )
@@
     (in_bom no) (on_board yes)
     (property "Reference" "R702" (id 0) (at 170.18 69.85 90))
-    (property "Value" "" (id 1) (at 175.26 69.85 90))
-    (property "Footprint" "" (id 2) (at 173.736 70.104 90)
+    (property "Value" "200k" (id 1) (at 175.26 69.85 90))
+    (property "Footprint" "Resistor_SMD:R_0805_2012Metric" (id 2) (at 173.736 70.104 90)
       (effects (font (size 1.27 1.27)) hide)
     )
@@
     (in_bom no) (on_board yes)
     (property "Reference" "R703" (id 0) (at 170.18 77.47 90))
-    (property "Value" "" (id 1) (at 175.26 77.47 90))
-    (property "Footprint" "" (id 2) (at 173.736 77.724 90)
+    (property "Value" "120k" (id 1) (at 175.26 77.47 90))
+    (property "Footprint" "Resistor_SMD:R_0805_2012Metric" (id 2) (at 173.736 77.724 90)
       (effects (font (size 1.27 1.27)) hide)
     )
@@
       (effects (font (size 1.27 1.27)) (justify left))
     )
-    (property "Value" "" (id 1) (at 133.35 68.5799 0)
+    (property "Value" "1u" (id 1) (at 133.35 68.5799 0)
       (effects (font (size 1.27 1.27)) (justify left))
     )
-    (property "Footprint" "" (id 2) (at 130.5052 71.12 0)
+    (property "Footprint" "Capacitor_SMD:C_0805_2012Metric" (id 2) (at 130.5052 71.12 0)
       (effects (font (size 1.27 1.27)) hide)
     )
@@
     (in_bom yes) (on_board yes) (fields_autoplaced)
     (property "Reference" "U701" (id 0) (at 154.94 55.88 0))
-    (property "Value" "" (id 1) (at 154.94 58.42 0))
-    (property "Footprint" "" (id 2) (at 154.94 87.63 0)
+    (property "Value" "LP2951-3.3_SOIC" (id 1) (at 154.94 58.42 0))
+    (property "Footprint" "Package_SO:SOIC-8_3.9x4.9mm_P1.27mm" (id 2) (at 154.94 87.63 0)
       (effects (font (size 1.27 1.27)) hide)
     )
@@
     (in_bom no) (on_board yes)
     (property "Reference" "R701" (id 0) (at 138.43 76.2 90))
-    (property "Value" "" (id 1) (at 135.89 76.2 90))
-    (property "Footprint" "" (id 2) (at 143.256 76.454 90)
+    (property "Value" "10k" (id 1) (at 135.89 76.2 90))
+    (property "Footprint" "Resistor_SMD:R_0805_2012Metric" (id 2) (at 143.256 76.454 90)
       (effects (font (size 1.27 1.27)) hide)
     )
